File: hardware/prog_board/prog_board.sch (KiCad schematic (older format))
At the start: 15 parts, among them J1 USB_OTG, J2 Conn_01x06, Q1 MMBT2222, Q2 MMBT2222, U1 CP2104

Commit message: Working on schematic
Parts:
- removed J2: Conn_01x06, symbol Conn_01x06
- added J2: Conn_02x03_Odd_Even, symbol Conn_02x03_Odd_Even
- added SW1: SW_Push, footprint:KMR7, symbol SW_Push
- C2: value 4.7u -> 10u; footprint (none) -> Capacitors_SMD:C_0805; Part (none) -> 311-1460-1-ND; Source (none) -> DigiKey
Connections:
- wire segments 66 -> 61
Changed lines of the file:
@@
 NoConn ~ 4100 3700
 $Comp
-L Conn_01x06 J2
-U 1 1 5A4729E7
-P 9000 3000
-F 0 "J2" H 9000 3300 50  0000 C CNN
-F 1 "Conn_01x06" H 9000 2600 50  0000 C CNN
-F 2 "" H 9000 3000 50  0001 C CNN
-F 3 "" H 9000 3000 50  0001 C CNN
-	1    9000 3000
-	1    0    0    -1
-$EndComp
-$Comp
-L GND #PWR14
+L GND #PWR15
 U 1 1 5A472AC5
-P 8700 3400
-F 0 "#PWR14" H 8700 3150 50  0001 C CNN
-F 1 "GND" H 8700 3250 50  0000 C CNN
-F 2 "" H 8700 3400 50  0001 C CNN
-F 3 "" H 8700 3400 50  0001 C CNN
-	1    8700 3400
-	1    0    0    -1
-$EndComp
-$Comp
-L +5V #PWR13
+P 8900 3700
+F 0 "#PWR15" H 8900 3450 50  0001 C CNN
+F 1 "GND" H 8900 3550 50  0000 C CNN
+F 2 "" H 8900 3700 50  0001 C CNN
+F 3 "" H 8900 3700 50  0001 C CNN
+	1    8900 3700
+	1    0    0    -1
+$EndComp
+$Comp
+L +5V #PWR14
 U 1 1 5A472AEB
-P 8700 2700
-F 0 "#PWR13" H 8700 2550 50  0001 C CNN
-F 1 "+5V" H 8700 2840 50  0000 C CNN
-F 2 "" H 8700 2700 50  0001 C CNN
-F 3 "" H 8700 2700 50  0001 C CNN
-	1    8700 2700
-	1    0    0    -1
-$EndComp
-Text Label 8400 3000 0    60   ~ 0
+P 8200 3300
+F 0 "#PWR14" H 8200 3150 50  0001 C CNN
+F 1 "+5V" H 8200 3440 50  0000 C CNN
+F 2 "" H 8200 3300 50  0001 C CNN
+F 3 "" H 8200 3300 50  0001 C CNN
+	1    8200 3300
+	1    0    0    -1
+$EndComp
+Text Label 7950 3600 0    60   ~ 0
 GPIO0
-Text Label 8400 2900 0    60   ~ 0
+Text Label 7950 3500 0    60   ~ 0
 RESET
-Text Label 8400 3100 0    60   ~ 0
+Text Label 8850 3400 0    60   ~ 0
 TXD
-Text Label 8400 3200 0    60   ~ 0
+Text Label 8850 3500 0    60   ~ 0
 RXD
 $Comp
@@
 $EndComp
 $Comp
-L +3.3V #PWR12
+L +3.3V #PWR13
 U 1 1 5A4740AD
 P 6600 1650
-F 0 "#PWR12" H 6600 1500 50  0001 C CNN
+F 0 "#PWR13" H 6600 1500 50  0001 C CNN
 F 1 "+3.3V" H 6600 1790 50  0000 C CNN
 F 2 "" H 6600 1650 50  0001 C CNN
@@
 	6200 2500 6200 2400
 Wire Wire Line
-	8400 3200 8800 3200
-Wire Wire Line
-	8400 3100 8800 3100
-Wire Wire Line
-	8400 3000 8800 3000
-Wire Wire Line
-	8400 2900 8800 2900
-Wire Wire Line
-	8700 3300 8700 3400
-Wire Wire Line
-	8800 3300 8700 3300
-Wire Wire Line
-	8700 2800 8700 2700
-Wire Wire Line
-	8800 2800 8700 2800
+	8800 3500 9200 3500
+Wire Wire Line
+	8800 3400 9200 3400
+Wire Wire Line
+	7900 3600 8300 3600
+Wire Wire Line
+	7900 3500 8300 3500
+Wire Wire Line
+	8900 3600 8900 3700
+Wire Wire Line
+	8200 3400 8200 3300
+Wire Wire Line
+	8300 3400 8200 3400
 Connection ~ 3050 2900
 Wire Wire Line
@@
 Connection ~ 4000 2000
 Wire Wire Line
-	4000 1900 4000 2000
-Wire Wire Line
-	4000 2000 4000 2100
+	4000 1900 4000 2100
 Wire Wire Line
 	4000 2100 4100 2100
@@
 	3700 2200 3700 2300
 Wire Wire Line
-	3450 2200 3700 2200
-Wire Wire Line
-	3700 2200 4100 2200
-Wire Wire Line
-	3450 2900 3050 2900
-Wire Wire Line
-	3050 2900 2950 2900
-Wire Wire Line
-	3450 2200 3450 2900
-Wire Wire Line
-	3450 2900 3450 3000
+	3450 2200 4100 2200
+Wire Wire Line
+	2950 2900 3450 2900
+Wire Wire Line
+	3450 2200 3450 3000
 Wire Wire Line
 	3450 3000 4100 3000
@@
 	4100 2600 4000 2600
 Wire Wire Line
-	4000 2500 4000 2600
-Wire Wire Line
-	4000 2600 4000 2700
+	4000 2500 4000 2700
 Wire Wire Line
 	4100 2500 4000 2500
@@
 	4650 4800 4650 4700
 Wire Wire Line
-	3550 5700 3850 5700
-Wire Wire Line
-	3850 5700 3950 5700
+	3550 5700 3950 5700
 Wire Wire Line
 	3850 5400 3850 5700
@@
 	3850 5300 3850 5000
 Wire Wire Line
-	3550 5000 3850 5000
-Wire Wire Line
-	3850 5000 3950 5000
+	3550 5000 3950 5000
 Wire Wire Line
 	4350 5000 4250 5000
@@
 P 3050 1950
 F 0 "C2" H 3075 2050 50  0000 L CNN
-F 1 "4.7u" H 3075 1850 50  0000 L CNN
-F 2 "" H 3088 1800 50  0001 C CNN
+F 1 "10u" H 3075 1850 50  0000 L CNN
+F 2 "Capacitors_SMD:C_0805" H 3088 1800 50  0001 C CNN
 F 3 "" H 3050 1950 50  0001 C CNN
+F 4 "DigiKey" H 3050 1950 60  0001 C CNN "Source"
+F 5 "311-1460-1-ND" H 3050 1950 60  0001 C CNN "Part"
 	1    3050 1950
 	1    0    0    -1
@@
 Wire Wire Line
 	3800 3400 3800 3450
+$Comp
+L Conn_02x03_Odd_Even J2
+U 1 1 5A47BEAC
+P 8500 3500
+F 0 "J2" H 8550 3700 50  0000 C CNN
+F 1 "Conn_02x03_Odd_Even" H 8550 3300 50  0001 C CNN
+F 2 "" H 8500 3500 50  0001 C CNN
+F 3 "" H 8500 3500 50  0001 C CNN
+F 4 "DigiKey" H 8500 3500 60  0001 C CNN "Source"
+F 5 "S2111E-03-ND" H 8500 3500 60  0001 C CNN "Part"
+	1    8500 3500
+	1    0    0    -1
+$EndComp
+Wire Wire Line
+	8900 3600 8800 3600
+$Comp
+L SW_Push SW1
+U 1 1 5A47DA0C
+P 6400 5250
+F 0 "SW1" H 6450 5350 50  0000 L CNN
+F 1 "SW_Push" H 6400 5190 50  0001 C CNN
+F 2 "footprint:KMR7" H 6400 5450 50  0001 C CNN
+F 3 "" H 6400 5450 50  0001 C CNN
+F 4 "DigiKey" H 6400 5250 60  0001 C CNN "Source"
+F 5 "CKN10689CT-ND" H 6400 5250 60  0001 C CNN "Part"
+	1    6400 5250
+	0    -1   1    0
+$EndComp
+$Comp
+L GND #PWR12
+U 1 1 5A47DAFE
+P 6400 5550
+F 0 "#PWR12" H 6400 5300 50  0001 C CNN
+F 1 "GND" H 6400 5400 50  0000 C CNN
+F 2 "" H 6400 5550 50  0001 C CNN
+F 3 "" H 6400 5550 50  0001 C CNN
+	1    6400 5550
+	1    0    0    -1
+$EndComp
+Wire Wire Line
+	6400 5450 6400 5550
+Text Label 6400 4950 1    60   ~ 0
+RESET
+Wire Wire Line
+	6400 4650 6400 5050
 $EndSCHEMATC

Commit message: Working on layout
Parts:
- C4: footprint (none) -> Capacitors_SMD:C_0603; Part (none) -> 311-1455-1-ND; Source (none) -> DigiKey
- D1: Part (none) -> 160-1447-1-ND
- D2: Part (none) -> 160-1435-1-ND
- J1: footprint (none) -> footprint:10118192; Part (none) -> 609-4613-1-ND; Source (none) -> DigiKey
- J2: footprint (none) -> Pin_Headers:Pin_Header_Angled_2x03_Pitch2.54mm
Other:
- moved on the sheet: SW1
Changed lines of the file:
@@
 encoding utf-8
 Sheet 1 1
-Title ""
+Title "Wifi Hydrometer - Programmer Board"
 Date ""
-Rev ""
+Rev "2.0"
 Comp ""
 Comment1 ""
@@
 F 0 "J1" H 2450 3550 50  0000 L CNN
 F 1 "USB_OTG" H 2450 3450 50  0000 L CNN
-F 2 "" H 2800 3050 50  0001 C CNN
+F 2 "footprint:10118192" H 2800 3050 50  0001 C CNN
 F 3 "" H 2800 3050 50  0001 C CNN
+F 4 "DigiKey" H 2650 3100 60  0001 C CNN "Source"
+F 5 "609-4613-1-ND" H 2650 3100 60  0001 C CNN "Part"
 	1    2650 3100
 	1    0    0    -1
@@
 $EndComp
 $Comp
-L GND #PWR10
+L GND #PWR01
 U 1 1 5A471622
 P 4000 2700
-F 0 "#PWR10" H 4000 2450 50  0001 C CNN
+F 0 "#PWR01" H 4000 2450 50  0001 C CNN
 F 1 "GND" H 4000 2550 50  0000 C CNN
 F 2 "" H 4000 2700 50  0001 C CNN
@@
 $EndComp
 $Comp
-L GND #PWR1
+L GND #PWR02
 U 1 1 5A4716B6
 P 2650 3600
-F 0 "#PWR1" H 2650 3350 50  0001 C CNN
+F 0 "#PWR02" H 2650 3350 50  0001 C CNN
 F 1 "GND" H 2650 3450 50  0000 C CNN
 F 2 "" H 2650 3600 50  0001 C CNN
@@
 RXD
 $Comp
-L GND #PWR7
+L GND #PWR03
 U 1 1 5A471B3F
 P 3700 2700
-F 0 "#PWR7" H 3700 2450 50  0001 C CNN
+F 0 "#PWR03" H 3700 2450 50  0001 C CNN
 F 1 "GND" H 3700 2550 50  0000 C CNN
 F 2 "" H 3700 2700 50  0001 C CNN
@@
 $EndComp
 $Comp
-L GND #PWR3
+L GND #PWR04
 U 1 1 5A471D5B
 P 2750 2200
-F 0 "#PWR3" H 2750 1950 50  0001 C CNN
+F 0 "#PWR04" H 2750 1950 50  0001 C CNN
 F 1 "GND" H 2750 2050 50  0000 C CNN
 F 2 "" H 2750 2200 50  0001 C CNN
@@
 $EndComp
 $Comp
-L +3.3V #PWR9
+L +3.3V #PWR05
 U 1 1 5A471FDB
 P 4000 1900
-F 0 "#PWR9" H 4000 1750 50  0001 C CNN
+F 0 "#PWR05" H 4000 1750 50  0001 C CNN
 F 1 "+3.3V" H 4000 2040 50  0000 C CNN
 F 2 "" H 4000 1900 50  0001 C CNN
@@
 $EndComp
 $Comp
-L +3.3V #PWR2
+L +3.3V #PWR06
 U 1 1 5A4720E8
 P 2750 1700
-F 0 "#PWR2" H 2750 1550 50  0001 C CNN
+F 0 "#PWR06" H 2750 1550 50  0001 C CNN
 F 1 "+3.3V" H 2750 1840 50  0000 C CNN
 F 2 "" H 2750 1700 50  0001 C CNN
@@
 $EndComp
 $Comp
-L +5V #PWR6
+L +5V #PWR07
 U 1 1 5A472647
 P 3050 2800
-F 0 "#PWR6" H 3050 2650 50  0001 C CNN
+F 0 "#PWR07" H 3050 2650 50  0001 C CNN
 F 1 "+5V" H 3050 2940 50  0000 C CNN
 F 2 "" H 3050 2800 50  0001 C CNN
@@
 NoConn ~ 4100 3700
 $Comp
-L GND #PWR15
+L GND #PWR08
 U 1 1 5A472AC5
 P 8900 3700
-F 0 "#PWR15" H 8900 3450 50  0001 C CNN
+F 0 "#PWR08" H 8900 3450 50  0001 C CNN
 F 1 "GND" H 8900 3550 50  0000 C CNN
 F 2 "" H 8900 3700 50  0001 C CNN
@@
 $EndComp
 $Comp
-L +5V #PWR14
+L +5V #PWR09
 U 1 1 5A472AEB
 P 8200 3300
-F 0 "#PWR14" H 8200 3150 50  0001 C CNN
+F 0 "#PWR09" H 8200 3150 50  0001 C CNN
 F 1 "+5V" H 8200 3440 50  0000 C CNN
 F 2 "" H 8200 3300 50  0001 C CNN
@@
 F 3 "" H 6200 2250 50  0001 C CNN
 F 4 "DigiKey" H 6200 2250 60  0001 C CNN "Source"
+F 5 "160-1447-1-ND" H 6200 2250 60  0001 C CNN "Part"
 	1    6200 2250
 	0    -1   -1   0
@@
 F 3 "" H 6600 2250 50  0001 C CNN
 F 4 "DigiKey" H 6600 2250 60  0001 C CNN "Source"
+F 5 "160-1435-1-ND" H 6600 2250 60  0001 C CNN "Part"
 	1    6600 2250
 	0    -1   -1   0
 $EndComp
 $Comp
-L +3.3V #PWR13
+L +3.3V #PWR010
 U 1 1 5A4740AD
 P 6600 1650
-F 0 "#PWR13" H 6600 1500 50  0001 C CNN
+F 0 "#PWR010" H 6600 1500 50  0001 C CNN
 F 1 "+3.3V" H 6600 1790 50  0000 C CNN
 F 2 "" H 6600 1650 50  0001 C CNN
@@
 $EndComp
 $Comp
-L +3.3V #PWR11
+L +3.3V #PWR011
 U 1 1 5A4742C2
 P 6200 1650
-F 0 "#PWR11" H 6200 1500 50  0001 C CNN
+F 0 "#PWR011" H 6200 1500 50  0001 C CNN
 F 1 "+3.3V" H 6200 1790 50  0000 C CNN
 F 2 "" H 6200 1650 50  0001 C CNN
@@
 $EndComp
 $Comp
-L GND #PWR5
+L GND #PWR012
 U 1 1 5A475D01
 P 3050 2200
-F 0 "#PWR5" H 3050 1950 50  0001 C CNN
+F 0 "#PWR012" H 3050 1950 50  0001 C CNN
 F 1 "GND" H 3050 2050 50  0000 C CNN
 F 2 "" H 3050 2200 50  0001 C CNN
@@
 	3050 2100 3050 2200
 $Comp
-L +3.3V #PWR4
+L +3.3V #PWR013
 U 1 1 5A475DB7
 P 3050 1700
-F 0 "#PWR4" H 3050 1550 50  0001 C CNN
+F 0 "#PWR013" H 3050 1550 50  0001 C CNN
 F 1 "+3.3V" H 3050 1840 50  0000 C CNN
 F 2 "" H 3050 1700 50  0001 C CNN
@@
 F 0 "C4" H 3825 3700 50  0000 L CNN
 F 1 "4.7u" H 3825 3500 50  0000 L CNN
-F 2 "" H 3838 3450 50  0001 C CNN
+F 2 "Capacitors_SMD:C_0603" H 3838 3450 50  0001 C CNN
 F 3 "" H 3800 3600 50  0001 C CNN
+F 4 "DigiKey" H 3800 3600 60  0001 C CNN "Source"
+F 5 "311-1455-1-ND" H 3800 3600 60  0001 C CNN "Part"
 	1    3800 3600
 	1    0    0    -1
 $EndComp
 $Comp
-L GND #PWR8
+L GND #PWR014
 U 1 1 5A4762F2
 P 3800 3800
-F 0 "#PWR8" H 3800 3550 50  0001 C CNN
+F 0 "#PWR014" H 3800 3550 50  0001 C CNN
 F 1 "GND" H 3800 3650 50  0000 C CNN
 F 2 "" H 3800 3800 50  0001 C CNN
@@
 F 0 "J2" H 8550 3700 50  0000 C CNN
 F 1 "Conn_02x03_Odd_Even" H 8550 3300 50  0001 C CNN
-F 2 "" H 8500 3500 50  0001 C CNN
+F 2 "Pin_Headers:Pin_Header_Angled_2x03_Pitch2.54mm" H 8500 3500 50  0001 C CNN
 F 3 "" H 8500 3500 50  0001 C CNN
 F 4 "DigiKey" H 8500 3500 60  0001 C CNN "Source"
@@
 L SW_Push SW1
 U 1 1 5A47DA0C
-P 6400 5250
-F 0 "SW1" H 6450 5350 50  0000 L CNN
-F 1 "SW_Push" H 6400 5190 50  0001 C CNN
-F 2 "footprint:KMR7" H 6400 5450 50  0001 C CNN
-F 3 "" H 6400 5450 50  0001 C CNN
-F 4 "DigiKey" H 6400 5250 60  0001 C CNN "Source"
-F 5 "CKN10689CT-ND" H 6400 5250 60  0001 C CNN "Part"
-	1    6400 5250
+P 2450 5400
+F 0 "SW1" H 2500 5500 50  0000 L CNN
+F 1 "SW_Push" H 2450 5340 50  0001 C CNN
+F 2 "footprint:KMR7" H 2450 5600 50  0001 C CNN
+F 3 "" H 2450 5600 50  0001 C CNN
+F 4 "DigiKey" H 2450 5400 60  0001 C CNN "Source"
+F 5 "CKN10689CT-ND" H 2450 5400 60  0001 C CNN "Part"
+	1    2450 5400
 	0    -1   1    0
 $EndComp
 $Comp
-L GND #PWR12
+L GND #PWR015
 U 1 1 5A47DAFE
-P 6400 5550
-F 0 "#PWR12" H 6400 5300 50  0001 C CNN
-F 1 "GND" H 6400 5400 50  0000 C CNN
-F 2 "" H 6400 5550 50  0001 C CNN
-F 3 "" H 6400 5550 50  0001 C CNN
-	1    6400 5550
-	1    0    0    -1
-$EndComp
-Wire Wire Line
-	6400 5450 6400 5550
-Text Label 6400 4950 1    60   ~ 0
+P 2450 5700
+F 0 "#PWR015" H 2450 5450 50  0001 C CNN
+F 1 "GND" H 2450 5550 50  0000 C CNN
+F 2 "" H 2450 5700 50  0001 C CNN
+F 3 "" H 2450 5700 50  0001 C CNN
+	1    2450 5700
+	1    0    0    -1
+$EndComp
+Wire Wire Line
+	2450 5600 2450 5700
+Text Label 2450 5100 1    60   ~ 0
 RESET
 Wire Wire Line
-	6400 4650 6400 5050
+	2450 4800 2450 5200
 $EndSCHEMATC
