File: hardware/main_board/main_board.sch (KiCad schematic (older format))
At the start: 33 parts, among them J1 eConn_02x03_Odd_Even, P1 CONN_01X02, Q1 DMG3415U, SW1 SW_DPDT_x2, U1 MCP73831/2, U2 AP2112, U3 Si1145, U4 MCP9808, U5 ESP-WROOM-32D, U6 MMA8451Q

Commit message: Minor changes to BOM
Parts:
- R8: Part 311-2.00KHRCT-ND -> 311-10.0KHRCT-ND
- U5: Part (none) -> 1528-1801-ND
Other:
- note added: "ADDR: 0x18"
- note added: "ADDR: 0x1D"
- note added: "ADDR: 0x60"
